File: Labs/Lab2/report/seven_segment_all.sch (EAGLE design)
At the start: 32 parts, among them Q1 2N3906, Q2 2N3906

Commit message: Finished lab report 2
Changed lines of the file:
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@@
 </classes>
 <parts>
-<part name="PIN1" library="supply2" deviceset="V--&gt;" device="" value="s[1] / P1"/>
+<part name="PIN1" library="supply2" deviceset="V--&gt;" device="" value="s3[1] / P1"/>
 <part name="R1" library="resistor" deviceset="R-US_" device="0411/12" value="10k"/>
 <part name="R2" library="resistor" deviceset="R-US_" device="0411/12" value="220"/>
 <part name="B2" library="adafruit" deviceset="LED" device="5MM"/>
-<part name="PIN2" library="supply2" deviceset="V--&gt;" device="" value="s[0] / P2"/>
-<part name="PIN3" library="supply2" deviceset="V--&gt;" device="" value="s[5] / P3"/>
-<part name="PIN4" library="supply2" deviceset="V--&gt;" device="" value="s[2] / P4"/>
+<part name="PIN2" library="supply2" deviceset="V--&gt;" device="" value="s3[0] / P2"/>
+<part name="PIN3" library="supply2" deviceset="V--&gt;" device="" value="s3[5] / P3"/>
+<part name="PIN4" library="supply2" deviceset="V--&gt;" device="" value="s3[2] / P4"/>
 <part name="+3V4" library="supply1" deviceset="+3V3" device=""/>
-<part name="PIN5" library="supply2" deviceset="V--&gt;" device="" value="s[6] / P7"/>
-<part name="PIN6" library="supply2" deviceset="V--&gt;" device="" value="s[3] / P10"/>
-<part name="PIN11" library="supply2" deviceset="V--&gt;" device="" value="s[4] / P11"/>
+<part name="PIN5" library="supply2" deviceset="V--&gt;" device="" value="s3[6] / P7"/>
+<part name="PIN6" library="supply2" deviceset="V--&gt;" device="" value="s3[3] / P10"/>
+<part name="PIN11" library="supply2" deviceset="V--&gt;" device="" value="s3[4] / P11"/>
 <part name="Q1" library="transistor-pnp" deviceset="2N3906" device=""/>
 <part name="SUPPLY1" library="sherman" deviceset="V--&gt;" device="" value="on1 / P87"/>

Commit message: Started Lab3. Outlined code
Parts:
- added R17, R18: 10k, resistor:R-US_0411/12
Connections:
- new net N$12: R16.2, R18.1
- new net N$4: R15.2, R17.1
- net +3V3: now also R17.2, R18.2
Changed lines of the file:
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@@
 <part name="R15" library="resistor" deviceset="R-US_" device="0411/12" value="5.6k"/>
 <part name="R16" library="resistor" deviceset="R-US_" device="0411/12" value="5.6k"/>
+<part name="R17" library="resistor" deviceset="R-US_" device="0411/12" value="10k"/>
+<part name="R18" library="resistor" deviceset="R-US_" device="0411/12" value="10k"/>
+<part name="+3V10" library="supply1" deviceset="+3V3" device=""/>
+<part name="+3V11" library="supply1" deviceset="+3V3" device=""/>
 </parts>
 <sheets>
@@
 <instance part="PIN11" gate="G$1" x="177.8" y="22.86"/>
 <instance part="Q1" gate="G$1" x="83.82" y="66.04"/>
-<instance part="SUPPLY1" gate="G$1" x="71.12" y="66.04"/>
+<instance part="SUPPLY1" gate="G$1" x="60.96" y="66.04"/>
 <instance part="B1" gate="G$1" x="30.48" y="45.72"/>
 <instance part="+3V1" gate="G$1" x="12.7" y="45.72"/>
@@
 <instance part="+3V9" gate="G$1" x="132.08" y="83.82"/>
 <instance part="Q2" gate="G$1" x="129.54" y="66.04"/>
-<instance part="SUPPLY2" gate="G$1" x="116.84" y="66.04"/>
+<instance part="SUPPLY2" gate="G$1" x="106.68" y="66.04"/>
 <instance part="R15" gate="G$1" x="76.2" y="66.04" rot="R180"/>
 <instance part="R16" gate="G$1" x="121.92" y="66.04" rot="R180"/>
+<instance part="R17" gate="G$1" x="66.04" y="71.12" rot="R90"/>
+<instance part="R18" gate="G$1" x="111.76" y="71.12" rot="R90"/>
+<instance part="+3V10" gate="G$1" x="66.04" y="78.74"/>
+<instance part="+3V11" gate="G$1" x="111.76" y="78.74"/>
 </instances>
 <busses>
@@
 <pinref part="+3V9" gate="G$1" pin="+3V3"/>
 <wire x1="132.08" y1="71.12" x2="132.08" y2="81.28" width="0.1524" layer="91"/>
+</segment>
+<segment>
+<pinref part="R17" gate="G$1" pin="2"/>
+<pinref part="+3V10" gate="G$1" pin="+3V3"/>
+</segment>
+<segment>
+<pinref part="R18" gate="G$1" pin="2"/>
+<pinref part="+3V11" gate="G$1" pin="+3V3"/>
 </segment>
 </net>
@@
 </segment>
 </net>
+<net name="N$4" class="0">
+<segment>
+<pinref part="R15" gate="G$1" pin="2"/>
+<pinref part="R17" gate="G$1" pin="1"/>
+<wire x1="71.12" y1="66.04" x2="66.04" y2="66.04" width="0.1524" layer="91"/>
+<wire x1="66.04" y1="66.04" x2="60.96" y2="66.04" width="0.1524" layer="91"/>
+<junction x="66.04" y="66.04"/>
+</segment>
+</net>
+<net name="N$12" class="0">
+<segment>
+<pinref part="R16" gate="G$1" pin="2"/>
+<pinref part="R18" gate="G$1" pin="1"/>
+<wire x1="116.84" y1="66.04" x2="111.76" y2="66.04" width="0.1524" layer="91"/>
+<wire x1="111.76" y1="66.04" x2="106.68" y2="66.04" width="0.1524" layer="91"/>
+<junction x="111.76" y="66.04"/>
+</segment>
+</net>
